Commit message: modified urdf model files for tiny agent

File: Humanoid_Basic_Env/resources/tiny/tiny.urdf (robot description, URDF)
Before this commit: robot HumanoidTiny, 16 links, 15 joints
Links:
- removed link chest
- removed link left_ankle
- removed link left_elbow
- removed link left_hip
- removed link left_knee
- removed link left_shoulder
- removed link left_wrist
- removed link neck
- removed link right_ankle
- removed link right_elbow
- removed link right_knee
- removed link right_shoulder
- removed link right_wrist
Joints:
- removed joint chest
- removed joint left_ankle
- removed joint left_elbow
- removed joint left_hip
- removed joint left_knee
- removed joint left_shoulder
- removed joint left_wrist
- removed joint neck
- removed joint right_ankle
- removed joint right_elbow
- removed joint right_knee
- removed joint right_shoulder
- removed joint right_wrist

File: Humanoid_Basic_Env/resources/tiny/tinyTarget.urdf (robot description, URDF)
Before this commit: robot HumanoidTarget, 16 links, 15 joints
Links:
- removed link chest
- removed link left_ankle
- removed link left_elbow
- removed link left_hip
- removed link left_knee
- removed link left_shoulder
- removed link left_wrist
- removed link neck
- removed link right_ankle
- removed link right_elbow
- removed link right_knee
- removed link right_shoulder
- removed link right_wrist
Joints:
- removed joint chest
- removed joint left_ankle
- removed joint left_elbow
- removed joint left_hip
- removed joint left_knee
- removed joint left_shoulder
- removed joint left_wrist
- removed joint neck
- removed joint right_ankle
- removed joint right_elbow
- removed joint right_knee
- removed joint right_shoulder
- removed joint right_wrist
